File: PCBs/TheBrain/CM4_Module.kicad_sch (KiCad schematic)
At the start: 7 parts, among them U3 74LVC1G07SE-7

Commit message: Started Brain PCB
Parts:
- removed TP2: TestPoint, TestPoint:TestPoint_Pad_2.0x2.0mm, symbol Connector:TestPoint
Connections:
- net GLOBAL_EN: no longer names the net of Module1.99 (Global_EN)
- no-connect marks 117 -> 118
Changed lines of the file:
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@@
 	)
 	(junction
-		(at 149.86 49.657)
-		(diameter 1.016)
-		(color 0 0 0 0)
-	)
-	(junction
 		(at 187.96 142.24)
 		(diameter 1.016)
@@
 	)
 	(no_connect
+		(at 101.6 147.32)
+	)
+	(no_connect
 		(at 190.5 91.44)
 	)
@@
 	(wire
 		(pts
+			(xy 133.35 57.15) (xy 142.24 57.15)
+		)
+		(stroke
+			(width 0)
+			(type solid)
+		)
+	)
+	(wire
+		(pts
 			(xy 118.364 48.26) (xy 118.364 45.72)
 		)
@@
 	(wire
 		(pts
-			(xy 101.6 121.92) (xy 101.6 124.46)
+			(xy 34.29 121.92) (xy 40.64 121.92)
 		)
 		(stroke
@@
 	(wire
 		(pts
-			(xy 120.65 64.77) (xy 134.62 64.77)
+			(xy 101.6 121.92) (xy 101.6 124.46)
 		)
 		(stroke
@@
 	(wire
 		(pts
-			(xy 113.284 21.59) (xy 118.364 21.59)
+			(xy 113.03 21.59) (xy 118.364 21.59)
 		)
 		(stroke
@@
 	(wire
 		(pts
+			(xy 121.92 64.77) (xy 134.62 64.77)
+		)
+		(stroke
+			(width 0)
+			(type solid)
+		)
+	)
+	(wire
+		(pts
 			(xy 251.46 104.14) (xy 254 104.14)
 		)
@@
 	(wire
 		(pts
-			(xy 149.86 49.657) (xy 149.86 50.8)
+			(xy 149.86 49.53) (xy 149.86 50.8)
 		)
 		(stroke
@@
 	(wire
 		(pts
-			(xy 144.8562 49.657) (xy 149.86 49.657)
-		)
-		(stroke
-			(width 0)
-			(type solid)
-		)
-	)
-	(wire
-		(pts
 			(xy 39.37 104.14) (xy 40.64 104.14)
 		)
@@
 	(wire
 		(pts
-			(xy 35.56 121.92) (xy 40.64 121.92)
-		)
-		(stroke
-			(width 0)
-			(type solid)
-		)
-	)
-	(wire
-		(pts
 			(xy 254 111.76) (xy 254 119.38)
 		)
@@
 	(wire
 		(pts
+			(xy 34.29 124.46) (xy 40.64 124.46)
+		)
+		(stroke
+			(width 0)
+			(type solid)
+		)
+	)
+	(wire
+		(pts
 			(xy 187.96 66.04) (xy 187.96 73.66)
 		)
@@
 	(wire
 		(pts
-			(xy 142.24 57.15) (xy 133.35 57.15)
-		)
-		(stroke
-			(width 0)
-			(type solid)
-		)
-	)
-	(wire
-		(pts
 			(xy 101.6 38.1) (xy 102.87 38.1)
 		)
@@
 	(wire
 		(pts
-			(xy 101.6 147.32) (xy 107.95 147.32)
-		)
-		(stroke
-			(width 0)
-			(type solid)
-		)
-	)
-	(wire
-		(pts
 			(xy 22.86 127) (xy 40.64 127)
 		)
@@
 	(wire
 		(pts
-			(xy 35.56 124.46) (xy 40.64 124.46)
-		)
-		(stroke
-			(width 0)
-			(type solid)
-		)
-	)
-	(wire
-		(pts
 			(xy 40.64 38.1) (xy 39.37 38.1)
 		)
@@
 	(wire
 		(pts
-			(xy 149.86 49.53) (xy 149.86 49.657)
-		)
-		(stroke
-			(width 0)
-			(type solid)
-		)
-	)
-	(wire
-		(pts
 			(xy 190.5 149.86) (xy 187.96 149.86)
 		)
@@
 	)
 	(label "nPWR_LED"
-		(at 123.19 64.77 0)
+		(at 121.92 64.77 0)
 		(fields_autoplaced yes)
 		(effects
@@
 	)
 	(label "+3.3v"
-		(at 138.43 57.15 180)
+		(at 133.35 57.15 0)
 		(fields_autoplaced yes)
 		(effects
@@
 				(size 1.27 1.27)
 			)
-			(justify right bottom)
+			(justify left bottom)
 		)
 	)
@@
 	)
 	(label "+3.3v"
-		(at 118.364 21.59 180)
+		(at 22.86 127 0)
 		(fields_autoplaced yes)
 		(effects
@@
 				(size 1.27 1.27)
 			)
-			(justify right bottom)
+			(justify left bottom)
 		)
 	)
-	(label "+3.3v"
-		(at 22.86 127 0)
+	(label "+5v"
+		(at 107.95 119.38 180)
 		(fields_autoplaced yes)
 		(effects
@@
 				(size 1.27 1.27)
 			)
-			(justify left bottom)
+			(justify right bottom)
 		)
 	)
-	(label "+5v"
-		(at 107.95 119.38 180)
+	(label "+3.3v"
+		(at 113.03 21.59 0)
 		(fields_autoplaced yes)
 		(effects
@@
 				(size 1.27 1.27)
 			)
-			(justify right bottom)
+			(justify left bottom)
 		)
 	)
@@
 		)
 	)
+	(hierarchical_label "SCL0"
+		(shape output)
+		(at 34.29 121.92 180)
+		(fields_autoplaced yes)
+		(effects
+			(font
+				(size 1.27 1.27)
+			)
+			(justify right)
+		)
+	)
 	(hierarchical_label "HDMI0_SCL"
 		(shape input)
@@
 		)
 	)
-	(hierarchical_label "GLOBAL_EN"
-		(shape input)
-		(at 107.95 147.32 0)
-		(fields_autoplaced yes)
-		(effects
-			(font
-				(size 1.27 1.27)
-			)
-			(justify left)
-		)
-	)
 	(hierarchical_label "HDMI0_D0_N"
 		(shape input)
@@
 		)
 	)
-	(hierarchical_label "SCL0"
-		(shape output)
-		(at 35.56 121.92 180)
-		(fields_autoplaced yes)
-		(effects
-			(font
-				(size 1.27 1.27)
-			)
-			(justify right)
-		)
-	)
 	(hierarchical_label "HDMI0_D2_N"
 		(shape input)
@@
 		)
 	)
-	(hierarchical_label "SDA0"
-		(shape output)
-		(at 35.56 124.46 180)
-		(fields_autoplaced yes)
-		(effects
-			(font
-				(size 1.27 1.27)
-			)
-			(justify right)
-		)
-	)
 	(hierarchical_label "SDA1"
 		(shape input)
@@
 		)
 	)
+	(hierarchical_label "SDA0"
+		(shape output)
+		(at 34.29 124.46 180)
+		(fields_autoplaced yes)
+		(effects
+			(font
+				(size 1.27 1.27)
+			)
+			(justify right)
+		)
+	)
 	(symbol
 		(lib_id "CM4IO:ComputeModule4-CM4")
@@
 					(unit 1)
 				)
-			)
-		)
-	)
-	(symbol
-		(lib_id "Connector:TestPoint")
-		(at 144.8562 49.657 90)
-		(unit 1)
-		(exclude_from_sim no)
-		(in_bom yes)
-		(on_board yes)
-		(dnp no)
-		(property "Reference" "TP2"
-			(at 142.494 46.99 90)
-			(effects
-				(font
-					(size 1.27 1.27)
-				)
-				(justify left)
-			)
-		)
-		(property "Value" "TestPoint"
-			(at 147.574 52.07 90)
-			(effects
-				(font
-					(size 1.27 1.27)
-				)
-				(justify left)
-			)
-		)
-		(property "Footprint" "TestPoint:TestPoint_Pad_2.0x2.0mm"
-			(at 144.8562 44.577 0)
-			(effects
-				(font
-					(size 1.27 1.27)
-				)
-				(hide yes)
-			)
-		)
-		(property "Datasheet" ""
-			(at 144.8562 44.577 0)
-			(effects
-				(font
-					(size 1.27 1.27)
-				)
-				(hide yes)
-			)
-		)
-		(property "Description" ""
-			(at 144.8562 49.657 0)
-			(effects
-				(font
-					(size 1.27 1.27)
-				)
-				(hide yes)
-			)
-		)
-		(property "Field4" "nf"
-			(at 144.8562 49.657 0)
-			(effects
-				(font
-					(size 1.27 1.27)
-				)
-				(hide yes)
-			)
-		)
-		(property "Field5" "nf"
-			(at 144.8562 49.657 0)
-			(effects
-				(font
-					(size 1.27 1.27)
-				)
-				(hide yes)
-			)
-		)
-		(property "Field6" "nf"
-			(at 144.8562 49.657 0)
-			(effects
-				(font
-					(size 1.27 1.27)
-				)
-				(hide yes)
-			)
-		)
-		(property "Field7" "nf"
-			(at 144.8562 49.657 0)
-			(effects
-				(font
-					(size 1.27 1.27)
-				)
-				(hide yes)
-			)
-		)
-		(pin "1"
-		)
-		(instances
-			(project "TheBrain"
-				(path "/65a43853-fed5-47dc-8496-a0facecf291b/e01117e7-e4d0-4aaa-9507-8d22ff79cac6"
-					(reference "TP2")
-					(unit 1)
-				)
