File: PCBs/TheBrain/TheBrain.kicad_pcb (KiCad board)
At the start: 2 copper layers, 35 parts, among them J1 Molex 470531000, J2 690-019-298-412, J3 SM04B-SRSS-TB, J4 USB_A, U1 RT9742SNGV, U2 AP22653W6, U3 74LVC1G07SE-7, U4 PCF85063AT/AAZ, U5 EMC2301-1-ACZL-TR, U6 74LVC1G07SE-7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

Commit message: Started Brain PCB
Parts:
- removed BT1: Battery_Cell, Battery:BatteryHolder_Keystone_3034_1x20mm
- removed C11, C12, C9: 100n, Capacitor_SMD:C_0402_1005Metric
- removed D3: BAT54C-7-F, Package_TO_SOT_SMD:SOT-23
- removed R5, R6: 510K 1%, Resistor_SMD:R_0402_1005Metric
- removed TP2: TestPoint, TestPoint:TestPoint_Pad_2.0x2.0mm
- removed U4: PCF85063AT/AAZ, Package_SO:SOIC-8_3.9x4.9mm_P1.27mm
- removed U6: 74LVC1G07SE-7, Package_TO_SOT_SMD:SOT-353_SC-70-5
- removed Y1: X32K768S301, Crystal:Crystal_SMD_3215-2Pin_3.2x1.5mm
- moved R4 85.5 mm to (82.0, 80.8), turned to 90 degrees
- moved J3 84.0 mm to (82.6, 96.5), turned to 180 degrees
- moved C3 83.7 mm to (82.1, 73.5), turned to 90 degrees
- moved U2 82.9 mm to (87.6, 74.0)
- moved U5 80.8 mm to (86.7, 81.6), turned to 180 degrees
- moved C7 76.6 mm to (85.1, 64.4), turned to 180 degrees
- moved C4 76.5 mm to (86.5, 68.4), turned to 180 degrees
- moved C8 76.0 mm to (85.1, 61.4), turned to 180 degrees
- moved R2 75.5 mm to (90.8, 73.7), turned to 90 degrees
- moved C10 75.4 mm to (91.4, 80.8), turned to 90 degrees
- moved C5 73.1 mm to (89.0, 61.4)
- moved C6 73.1 mm to (89.0, 64.4)
- moved J1 70.7 mm to (74.8, 84.2), turned to 90 degrees
- moved J4 61.8 mm to (84.6, 52.8), turned to 180 degrees
- moved U1 46.5 mm to (137.4, 88.0)
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Connections:
- net /RTC/SCL renamed /CM4 Module/SCL0
- net /RTC/SDA renamed /CM4 Module/SDA0
- Module1 pad 99: /RTC/GLOBAL_EN -> unconnected-(Module1A-Global_EN-Pad99)
Routing:
- net /+3.3V: track 0.00 -> 125.3 mm, vias 0 -> 9
- net /+5V: track 0.00 -> 90.7 mm
- net /CM4 Module/USB2_P: track 0.00 -> 56.3 mm
- net /CM4 Module/USB2_N: track 0.00 -> 56.3 mm
- net /CM4 Module/nPWR_LED: track 0.00 -> 53.7 mm, vias 0 -> 2
- net Net-(Module1A-PI_nLED_Activity): track 0.00 -> 44.3 mm, vias 0 -> 2
- net /Connectors/VBUS: track 0.00 -> 29.6 mm, vias 0 -> 2
- net /CM4 Module/HDMI0_D2_P: track 0.00 -> 28.4 mm
- net /CM4 Module/HDMI0_D2_N: track 0.00 -> 28.4 mm
- net /CM4 Module/SDA1: track 0.00 -> 27.8 mm, vias 0 -> 2
- net /CM4 Module/SDC1: track 0.00 -> 27.4 mm, vias 0 -> 2
- net /CM4 Module/HDMI0_CEC: track 0.00 -> 27.0 mm, vias 0 -> 2
- net /CM4 Module/HDMI0_D1_P: track 0.00 -> 26.2 mm
- net /CM4 Module/HDMI0_D1_N: track 0.00 -> 26.1 mm
- net /CM4 Module/HDMI0_HOTPLUG: track 0.00 -> 24.7 mm, vias 0 -> 2
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- added copper zone on B.Cu, net GND
- added copper zone on F.Cu, net GND
