File: PCBs/TheBrain/TheBrain.kicad_sch (KiCad schematic)
At the start: 0 parts

Commit message: Started Brain PCB
Other:
- sheet RTC renamed FanControl
- sheet CM4 Module ports: added none; removed GLOBAL_EN
- sheet FanControl: file RTC.kicad_sch -> FanControl.kicad_sch
- sheet FanControl ports: added none; removed GLOBAL_EN
Changed lines of the file:
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@@
+	(wire
+		(pts
+			(xy 76.2 114.3) (xy 76.2 138.43)
+		)
+		(stroke
+			(width 0)
+			(type default)
+		)
+	)
 	(wire
 		(pts
@@
 	(wire
 		(pts
-			(xy 77.47 114.3) (xy 77.47 138.43)
-		)
-		(stroke
-			(width 0)
-			(type default)
-		)
-	)
-	(wire
-		(pts
 			(xy 199.39 45.72) (xy 204.47 45.72)
 		)
@@
 	(wire
 		(pts
+			(xy 73.66 114.3) (xy 73.66 138.43)
+		)
+		(stroke
+			(width 0)
+			(type default)
+		)
+	)
+	(wire
+		(pts
 			(xy 101.6 71.12) (xy 143.51 71.12)
 		)
@@
 		(pts
 			(xy 101.6 77.47) (xy 143.51 77.47)
-		)
-		(stroke
-			(width 0)
-			(type default)
-		)
-	)
-	(wire
-		(pts
-			(xy 72.39 114.3) (xy 72.39 138.43)
-		)
-		(stroke
-			(width 0)
-			(type default)
-		)
-	)
-	(wire
-		(pts
-			(xy 69.85 114.3) (xy 69.85 138.43)
 		)
 		(stroke
@@
 			(color 0 0 0 0.0000)
 		)
-		(property "Sheetname" "RTC"
+		(property "Sheetname" "FanControl"
 			(at 41.91 137.7184 0)
 			(effects
@@
 			)
 		)
-		(property "Sheetfile" "RTC.kicad_sch"
+		(property "Sheetfile" "FanControl.kicad_sch"
 			(at 41.91 180.9246 0)
 			(effects
@@
 				)
 				(justify left top)
-			)
-		)
-		(pin "SCL" input
-			(at 69.85 138.43 90)
-			(effects
-				(font
-					(size 1.27 1.27)
-				)
-				(justify right)
-			)
-		)
-		(pin "SDA" input
-			(at 72.39 138.43 90)
-			(effects
-				(font
-					(size 1.27 1.27)
-				)
-				(justify right)
 			)
 		)
@@
 			)
 		)
-		(pin "GLOBAL_EN" output
-			(at 77.47 138.43 90)
-			(effects
-				(font
-					(size 1.27 1.27)
-				)
-				(justify right)
-			)
-		)
 		(pin "+3.3v" input
 			(at 41.91 149.86 180)
@@
 				)
 				(justify left)
+			)
+		)
+		(pin "SDA" input
+			(at 73.66 138.43 90)
+			(effects
+				(font
+					(size 1.27 1.27)
+				)
+				(justify right)
+			)
+		)
+		(pin "SCL" input
+			(at 76.2 138.43 90)
+			(effects
+				(font
+					(size 1.27 1.27)
+				)
+				(justify right)
 			)
 		)
@@
 			)
 		)
-		(pin "SCL0" output
-			(at 69.85 114.3 270)
-			(effects
-				(font
-					(size 1.27 1.27)
-				)
-				(justify left)
-			)
-		)
-		(pin "SDA0" output
-			(at 72.39 114.3 270)
-			(effects
-				(font
-					(size 1.27 1.27)
-				)
-				(justify left)
-			)
-		)
 		(pin "+3.3v" output
 			(at 40.64 48.26 180)
@@
 			)
 		)
-		(pin "GLOBAL_EN" input
-			(at 77.47 114.3 270)
-			(effects
-				(font
-					(size 1.27 1.27)
-				)
-				(justify left)
-			)
-		)
 		(pin "USB2_N" bidirectional
 			(at 101.6 63.5 0)
@@
 			)
 		)
+		(pin "SDA0" output
+			(at 73.66 114.3 270)
+			(effects
+				(font
+					(size 1.27 1.27)
+				)
+				(justify left)
+			)
+		)
+		(pin "SCL0" output
+			(at 76.2 114.3 270)
+			(effects
+				(font
+					(size 1.27 1.27)
+				)
+				(justify left)
+			)
+		)
